Commit message: intial

File: examples/rimless_wheel/RimlessWheel.xacro (robot description, xacro)
@@ -1,6 +1,12 @@
 <?xml version="1.0"?>
+<<<<<<< HEAD
 <robot xmlns="https://drake.mit.edu"
  xmlns:xsi="http://www.w3.org/2001/XMLSchema-instance"
  xsi:schemaLocation="https://drake.mit.edu ../../doc/drakeURDF.xsd"
+=======
+<robot xmlns="http://drake.mit.edu"
+ xmlns:xsi="http://www.w3.org/2001/XMLSchema-instance"
+ xsi:schemaLocation="http://drake.mit.edu ../../doc/drakeURDF.xsd"
+>>>>>>> intial
  xmlns:xacro="http://ros.org/wiki/xacro" name="RimlessWheel">
   <xacro:property name="m" value="1" />

File: manipulation/models/iiwa_description/urdf/iiwa14.xacro (robot description, xacro)
@@ -1,8 +1,11 @@
 <?xml version="1.0"?>
 <robot xmlns:xacro="http://www.ros.org/wiki/xacro">
+<<<<<<< HEAD
   <!-- Provide additional material for the silver logo band. -->
   <material name="Silver">
     <color rgba="0.6 0.6 0.6 1.0"/>
   </material>
+=======
+>>>>>>> intial
   <!-- Import all Gazebo-customization elements, including Gazebo colors -->
   <xacro:include filename="$(find iiwa_description)/urdf/iiwa.gazebo.xacro" />
@@ -132,4 +135,5 @@
       </inertial>
       <visual>
+<<<<<<< HEAD
         <origin rpy="0 0 0" xyz="0 0 0"/>
         <geometry>
@@ -145,4 +149,12 @@
         <material name="Grey"/>
       </visual>
+=======
+        <origin xyz="0 0 0" rpy="0 0 0"/>
+        <geometry>
+          <mesh filename="../meshes/visual/link_2.obj"/>
+        </geometry>
+        <material name="Orange"/>
+      </visual>
+>>>>>>> intial
       <xacro:if value="${collision_type == 'mesh'}">
         <collision>
@@ -156,5 +168,9 @@
       <xacro:if value="${collision_type == 'primitive'}">
         <collision>
+<<<<<<< HEAD
           <origin rpy="1.570796326794897 0 0" xyz="0 0.056 0.035"/>
+=======
+          <origin rpy="1.57079632679 0 0" xyz="0 0.056 0.035"/>
+>>>>>>> intial
           <geometry>
             <cylinder radius="0.101" length="0.29"/>
@@ -192,4 +208,5 @@
         <material name="Grey"/>
       </visual>
+<<<<<<< HEAD
       <visual>
         <origin rpy="0 0 0" xyz="0 0 0"/>
@@ -206,4 +223,6 @@
         <material name="Silver"/>
       </visual>
+=======
+>>>>>>> intial
       <xacro:if value="${collision_type == 'mesh'}">
         <collision>
@@ -247,4 +266,5 @@
       </inertial>
       <visual>
+<<<<<<< HEAD
         <origin rpy="0 0 0" xyz="0 0 0"/>
         <geometry>
@@ -260,4 +280,12 @@
         <material name="Grey"/>
       </visual>
+=======
+        <origin xyz="0 0 0" rpy="0 0 0"/>
+        <geometry>
+          <mesh filename="../meshes/visual/link_4.obj"/>
+        </geometry>
+        <material name="Orange"/>
+      </visual>
+>>>>>>> intial
       <xacro:if value="${collision_type == 'mesh'}">
         <collision>
@@ -271,5 +299,9 @@
       <xacro:if value="${collision_type == 'primitive'}">
         <collision>
+<<<<<<< HEAD
           <origin rpy="1.570796326794897 0 0" xyz="0 0.056 0.025"/>
+=======
+          <origin rpy="1.57079632679 0 0" xyz="0 0.056 0.025"/>
+>>>>>>> intial
           <geometry>
             <cylinder radius="0.092" length="0.25"/>
@@ -307,4 +339,5 @@
         <material name="Grey"/>
       </visual>
+<<<<<<< HEAD
       <visual>
         <origin rpy="0 0 0" xyz="0 0 0"/>
@@ -321,4 +354,6 @@
         <material name="Silver"/>
       </visual>
+=======
+>>>>>>> intial
       <xacro:if value="${collision_type == 'mesh'}">
         <collision>
@@ -362,4 +397,5 @@
       </inertial>
       <visual>
+<<<<<<< HEAD
         <origin rpy="0 0 0" xyz="0 0 0"/>
         <geometry>
@@ -372,4 +408,9 @@
         <geometry>
           <mesh filename="../meshes/visual/link_6_orange.obj"/>
+=======
+        <origin xyz="0 0 0" rpy="0 0 0"/>
+        <geometry>
+          <mesh filename="../meshes/visual/link_6.obj"/>
+>>>>>>> intial
         </geometry>
         <material name="Orange"/>
@@ -465,10 +506,18 @@
       <parent link="${robot_name}_link_7"/>
       <child link="${robot_name}_link_ee"/>
+<<<<<<< HEAD
       <origin rpy="0 -1.570796326794897 0" xyz="0 0 0.045"/>
+=======
+      <origin rpy="0 -1.57079632679 0" xyz="0 0 0.045"/>
+>>>>>>> intial
     </joint>
     <link name="${robot_name}_link_ee">
     </link>
     <frame name="${robot_name}_frame_ee" link="${robot_name}_link_ee"
+<<<<<<< HEAD
            xyz="0.09 0 0" rpy="3.141592653589793 0 1.570796326794897"/>
+=======
+           xyz="0.09 0 0" rpy="3.14159265359 0 1.57079632679"/>
+>>>>>>> intial
     <!--Extensions -->
     <xacro:iiwa_gazebo robot_name="${robot_name}" />

Commit message: Revert "intial"
This reverts commit 56f906021d206a2d940a31a804b60b813b6ab099.

File: examples/rimless_wheel/RimlessWheel.xacro (robot description, xacro)
@@ -1,12 +1,6 @@
 <?xml version="1.0"?>
-<<<<<<< HEAD
 <robot xmlns="https://drake.mit.edu"
  xmlns:xsi="http://www.w3.org/2001/XMLSchema-instance"
  xsi:schemaLocation="https://drake.mit.edu ../../doc/drakeURDF.xsd"
-=======
-<robot xmlns="http://drake.mit.edu"
- xmlns:xsi="http://www.w3.org/2001/XMLSchema-instance"
- xsi:schemaLocation="http://drake.mit.edu ../../doc/drakeURDF.xsd"
->>>>>>> intial
  xmlns:xacro="http://ros.org/wiki/xacro" name="RimlessWheel">
   <xacro:property name="m" value="1" />

File: manipulation/models/iiwa_description/urdf/iiwa14.xacro (robot description, xacro)
@@ -1,11 +1,8 @@
 <?xml version="1.0"?>
 <robot xmlns:xacro="http://www.ros.org/wiki/xacro">
-<<<<<<< HEAD
   <!-- Provide additional material for the silver logo band. -->
   <material name="Silver">
     <color rgba="0.6 0.6 0.6 1.0"/>
   </material>
-=======
->>>>>>> intial
   <!-- Import all Gazebo-customization elements, including Gazebo colors -->
   <xacro:include filename="$(find iiwa_description)/urdf/iiwa.gazebo.xacro" />
@@ -135,5 +132,4 @@
       </inertial>
       <visual>
-<<<<<<< HEAD
         <origin rpy="0 0 0" xyz="0 0 0"/>
         <geometry>
@@ -149,12 +145,4 @@
         <material name="Grey"/>
       </visual>
-=======
-        <origin xyz="0 0 0" rpy="0 0 0"/>
-        <geometry>
-          <mesh filename="../meshes/visual/link_2.obj"/>
-        </geometry>
-        <material name="Orange"/>
-      </visual>
->>>>>>> intial
       <xacro:if value="${collision_type == 'mesh'}">
         <collision>
@@ -168,9 +156,5 @@
       <xacro:if value="${collision_type == 'primitive'}">
         <collision>
-<<<<<<< HEAD
           <origin rpy="1.570796326794897 0 0" xyz="0 0.056 0.035"/>
-=======
-          <origin rpy="1.57079632679 0 0" xyz="0 0.056 0.035"/>
->>>>>>> intial
           <geometry>
             <cylinder radius="0.101" length="0.29"/>
@@ -208,5 +192,4 @@
         <material name="Grey"/>
       </visual>
-<<<<<<< HEAD
       <visual>
         <origin rpy="0 0 0" xyz="0 0 0"/>
@@ -223,6 +206,4 @@
         <material name="Silver"/>
       </visual>
-=======
->>>>>>> intial
       <xacro:if value="${collision_type == 'mesh'}">
         <collision>
@@ -266,5 +247,4 @@
       </inertial>
       <visual>
-<<<<<<< HEAD
         <origin rpy="0 0 0" xyz="0 0 0"/>
         <geometry>
@@ -280,12 +260,4 @@
         <material name="Grey"/>
       </visual>
-=======
-        <origin xyz="0 0 0" rpy="0 0 0"/>
-        <geometry>
-          <mesh filename="../meshes/visual/link_4.obj"/>
-        </geometry>
-        <material name="Orange"/>
-      </visual>
->>>>>>> intial
       <xacro:if value="${collision_type == 'mesh'}">
         <collision>
@@ -299,9 +271,5 @@
       <xacro:if value="${collision_type == 'primitive'}">
         <collision>
-<<<<<<< HEAD
           <origin rpy="1.570796326794897 0 0" xyz="0 0.056 0.025"/>
-=======
-          <origin rpy="1.57079632679 0 0" xyz="0 0.056 0.025"/>
->>>>>>> intial
           <geometry>
             <cylinder radius="0.092" length="0.25"/>
@@ -339,5 +307,4 @@
         <material name="Grey"/>
       </visual>
-<<<<<<< HEAD
       <visual>
         <origin rpy="0 0 0" xyz="0 0 0"/>
@@ -354,6 +321,4 @@
         <material name="Silver"/>
       </visual>
-=======
->>>>>>> intial
       <xacro:if value="${collision_type == 'mesh'}">
         <collision>
@@ -397,5 +362,4 @@
       </inertial>
       <visual>
-<<<<<<< HEAD
         <origin rpy="0 0 0" xyz="0 0 0"/>
         <geometry>
@@ -408,9 +372,4 @@
         <geometry>
           <mesh filename="../meshes/visual/link_6_orange.obj"/>
-=======
-        <origin xyz="0 0 0" rpy="0 0 0"/>
-        <geometry>
-          <mesh filename="../meshes/visual/link_6.obj"/>
->>>>>>> intial
         </geometry>
         <material name="Orange"/>
@@ -506,18 +465,10 @@
       <parent link="${robot_name}_link_7"/>
       <child link="${robot_name}_link_ee"/>
-<<<<<<< HEAD
       <origin rpy="0 -1.570796326794897 0" xyz="0 0 0.045"/>
-=======
-      <origin rpy="0 -1.57079632679 0" xyz="0 0 0.045"/>
->>>>>>> intial
     </joint>
     <link name="${robot_name}_link_ee">
     </link>
     <frame name="${robot_name}_frame_ee" link="${robot_name}_link_ee"
-<<<<<<< HEAD
            xyz="0.09 0 0" rpy="3.141592653589793 0 1.570796326794897"/>
-=======
-           xyz="0.09 0 0" rpy="3.14159265359 0 1.57079632679"/>
->>>>>>> intial
     <!--Extensions -->
     <xacro:iiwa_gazebo robot_name="${robot_name}" />
